Commit message: Fixed various issues when running the G1 simulation in Mujoco

File: assets/g1_dex3_sim/urdf/g1_29dof_with_hand_rev_1_0.urdf (robot description, URDF)
Before this commit: robot g1_29dof_with_hand_rev_1_0, 53 links, 52 joints
Links:
- link head_link: geometry collision mesh filename=../meshes/head_link.STL; visual mesh filename=../meshes/head_link.STL
- link left_ankle_pitch_link: geometry collision mesh filename=../meshes/left_ankle_pitch_link.STL; visual mesh filename=../meshes/left_ankle_pitch_link.STL
- link left_ankle_roll_link: geometry collision sphere radius=0.005; collision sphere radius=0.005
- link left_elbow_link: geometry collision mesh filename=../meshes/left_elbow_link.STL; visual mesh filename=../meshes/left_elbow_link.STL
- link left_hand_index_0_link: geometry collision mesh filename=../meshes/left_hand_index_0_link.STL; visual mesh filename=../meshes/left_hand_index_0_link.STL
- link left_hand_index_1_link: geometry collision mesh filename=../meshes/left_hand_index_1_link.STL; visual mesh filename=../meshes/left_hand_index_1_link.STL
- link left_hand_middle_0_link: geometry collision mesh filename=../meshes/left_hand_middle_0_link.STL; visual mesh filename=../meshes/left_hand_middle_0_link.STL
- link left_hand_middle_1_link: geometry collision mesh filename=../meshes/left_hand_middle_1_link.STL; visual mesh filename=../meshes/left_hand_middle_1_link.STL
- link left_hand_palm_link: geometry collision mesh filename=../meshes/left_hand_palm_link.STL; visual mesh filename=../meshes/left_hand_palm_link.STL
- link left_hand_thumb_0_link: geometry collision mesh filename=../meshes/left_hand_thumb_0_link.STL; visual mesh filename=../meshes/left_hand_thumb_0_link.STL
- link left_hand_thumb_1_link: geometry collision box size=0.02 0.03 0.02; visual mesh filename=../meshes/left_hand_thumb_1_link.STL
- link left_hand_thumb_2_link: geometry collision mesh filename=../meshes/left_hand_thumb_2_link.STL; visual mesh filename=../meshes/left_hand_thumb_2_link.STL
- link left_hip_pitch_link: geometry collision mesh filename=../meshes/left_hip_pitch_link.STL; visual mesh filename=../meshes/left_hip_pitch_link.STL
- link left_hip_roll_link: geometry collision mesh filename=../meshes/left_hip_roll_link.STL; visual mesh filename=../meshes/left_hip_roll_link.STL
- link left_hip_yaw_link: geometry collision mesh filename=../meshes/left_hip_yaw_link.STL; visual mesh filename=../meshes/left_hip_yaw_link.STL
- link left_knee_link: geometry collision mesh filename=../meshes/left_knee_link.STL; visual mesh filename=../meshes/left_knee_link.STL
- link left_shoulder_pitch_link: geometry collision cylinder length=0.05 radius=0.03; visual mesh filename=../meshes/left_shoulder_pitch_link.STL
- link left_shoulder_roll_link: geometry collision cylinder length=0.03 radius=0.03; visual mesh filename=../meshes/left_shoulder_roll_link.STL
- link left_shoulder_yaw_link: geometry collision mesh filename=../meshes/left_shoulder_yaw_link.STL; visual mesh filename=../meshes/left_shoulder_yaw_link.STL
- link left_wrist_pitch_link: geometry collision mesh filename=../meshes/left_wrist_pitch_link.STL; visual mesh filename=../meshes/left_wrist_pitch_link.STL
- link left_wrist_roll_link: geometry collision mesh filename=../meshes/left_wrist_roll_link.STL; visual mesh filename=../meshes/left_wrist_roll_link.STL
- link left_wrist_yaw_link: geometry collision mesh filename=../meshes/left_wrist_yaw_link.STL; visual mesh filename=../meshes/left_wrist_yaw_link.STL
- link logo_link: geometry collision mesh filename=../meshes/logo_link.STL; visual mesh filename=../meshes/logo_link.STL
- link pelvis: geometry visual mesh filename=../meshes/pelvis.STL
- link pelvis_contour_link: geometry collision mesh filename=../meshes/pelvis_contour_link.STL; visual mesh filename=../meshes/pelvis_contour_link.STL
- link right_ankle_pitch_link: geometry collision mesh filename=../meshes/right_ankle_pitch_link.STL; visual mesh filename=../meshes/right_ankle_pitch_link.STL
- link right_ankle_roll_link: geometry collision sphere radius=0.005; collision sphere radius=0.005
- link right_elbow_link: geometry collision mesh filename=../meshes/right_elbow_link.STL; visual mesh filename=../meshes/right_elbow_link.STL
- link right_hand_index_0_link: geometry collision mesh filename=../meshes/right_hand_index_0_link.STL; visual mesh filename=../meshes/right_hand_index_0_link.STL
- link right_hand_index_1_link: geometry collision mesh filename=../meshes/right_hand_index_1_link.STL; visual mesh filename=../meshes/right_hand_index_1_link.STL
- link right_hand_middle_0_link: geometry collision mesh filename=../meshes/right_hand_middle_0_link.STL; visual mesh filename=../meshes/right_hand_middle_0_link.STL
- link right_hand_middle_1_link: geometry collision mesh filename=../meshes/right_hand_middle_1_link.STL; visual mesh filename=../meshes/right_hand_middle_1_link.STL
- link right_hand_palm_link: geometry collision mesh filename=../meshes/right_hand_palm_link.STL; visual mesh filename=../meshes/right_hand_palm_link.STL
- link right_hand_thumb_0_link: geometry collision mesh filename=../meshes/right_hand_thumb_0_link.STL; visual mesh filename=../meshes/right_hand_thumb_0_link.STL
- link right_hand_thumb_1_link: geometry collision box size=0.02 0.03 0.02; visual mesh filename=../meshes/right_hand_thumb_1_link.STL
- link right_hand_thumb_2_link: geometry collision mesh filename=../meshes/right_hand_thumb_2_link.STL; visual mesh filename=../meshes/right_hand_thumb_2_link.STL
- link right_hip_pitch_link: geometry collision mesh filename=../meshes/right_hip_pitch_link.STL; visual mesh filename=../meshes/right_hip_pitch_link.STL
- link right_hip_roll_link: geometry collision mesh filename=../meshes/right_hip_roll_link.STL; visual mesh filename=../meshes/right_hip_roll_link.STL
- link right_hip_yaw_link: geometry collision mesh filename=../meshes/right_hip_yaw_link.STL; visual mesh filename=../meshes/right_hip_yaw_link.STL
- link right_knee_link: geometry collision mesh filename=../meshes/right_knee_link.STL; visual mesh filename=../meshes/right_knee_link.STL
- link right_shoulder_pitch_link: geometry collision cylinder length=0.05 radius=0.03; visual mesh filename=../meshes/right_shoulder_pitch_link.STL
- link right_shoulder_roll_link: geometry collision cylinder length=0.03 radius=0.03; visual mesh filename=../meshes/right_shoulder_roll_link.STL
- link right_shoulder_yaw_link: geometry collision mesh filename=../meshes/right_shoulder_yaw_link.STL; visual mesh filename=../meshes/right_shoulder_yaw_link.STL
- link right_wrist_pitch_link: geometry collision mesh filename=../meshes/right_wrist_pitch_link.STL; visual mesh filename=../meshes/right_wrist_pitch_link.STL
- link right_wrist_roll_link: geometry collision mesh filename=../meshes/right_wrist_roll_link.STL; visual mesh filename=../meshes/right_wrist_roll_link.STL
- link right_wrist_yaw_link: geometry collision mesh filename=../meshes/right_wrist_yaw_link.STL; visual mesh filename=../meshes/right_wrist_yaw_link.STL
- link torso_link: geometry collision mesh filename=../meshes/torso_link_rev_1_0.STL; visual mesh filename=../meshes/torso_link_rev_1_0.STL
- link waist_roll_link: geometry visual mesh filename=../meshes/waist_roll_link_rev_1_0.STL
- link waist_yaw_link: geometry visual mesh filename=../meshes/waist_yaw_link_rev_1_0.STL
